Commit message: Added assignment_2

File: platforms/ur5_ros2_gazebo/urdf/ur5.urdf.xacro (robot description, xacro)
@@ -89,5 +89,5 @@
     <visual>
       <geometry>
-        <mesh filename="$(find robotiq_85_description)/meshes/visual/ur_to_robotiq_adapter.dae" />
+        <mesh filename="file://$(find robotiq_85_description)/meshes/visual/ur_to_robotiq_adapter.dae" />
       </geometry>
       <material name="flat_black"/>
@@ -95,5 +95,5 @@
     <!--collision>
       <geometry>
-        <mesh filename="$(find robotiq_85_description)/meshes/collision/ur_to_robotiq_adapter.stl" />
+        <mesh filename="file://$(find robotiq_85_description)/meshes/collision/ur_to_robotiq_adapter.stl" />
       </geometry>
     </collision-->
